Commit message: done till basic behaviour tree with all plugins and its fully working exept behaviour tree need to configure and activate manualy

File: install/single_robo_discription/share/single_robo_discription/urdf/mobile_base.xacro (robot description, xacro)
@@ -115,15 +115,44 @@
                              o_xyz="0 0 0" o_rpy="0 0 0" />
     </link>
-     <!-- Front direction Link rod -->
+     <!-- Front direction Link rod
     <link name="front_direction_link_rod">
         <visual>
             <geometry>
-                <!-- <sphere radius="${wheel_radius / 2.0}" /> -->
-                <cylinder radius="${wheel_radius / 2.0}" length="${0.005}" />
-            </geometry>
-            <origin xyz="0 0 0" rpy="0 0 1.5708" />
-            <material name="grey" />
-        </visual>
-    </link>
+                <cylinder radius="${wheel_radius / 2.0}" length="${0.05}" />
+            </geometry>
+            <origin xyz="0 0 0" rpy="0 0 1.5708" />
+            <material name="grey" />
+        </visual>
+    </link>
+     Back direction Link rod
+    <link name="back_direction_link_rod">
+        <visual>
+            <geometry>
+                <cylinder radius="${wheel_radius / 2.0}" length="${0.05}" />
+            </geometry>
+            <origin xyz="0 0 0" rpy="0 0 1.5708" />
+            <material name="grey" />
+        </visual>
+    </link>
+    Left direction Link rod
+    <link name="left_direction_link_rod">
+        <visual>
+            <geometry>
+                <cylinder radius="${wheel_radius / 2.0}" length="${0.05}" />
+            </geometry>
+            <origin xyz="0 0 0" rpy="0 0 1.5708" />
+            <material name="grey" />
+        </visual>
+    </link>
+    Right direction Link rod
+    <link name="right_direction_link_rod">
+        <visual>
+            <geometry>
+                <cylinder radius="${wheel_radius / 2.0}" length="${0.05}" />
+            </geometry>
+            <origin xyz="0 0 0" rpy="0 0 1.5708" />
+            <material name="grey" />
+        </visual>
+    </link> -->
     <!-- Back Caster Wheel Link -->
     <link name="caster_wheel_link2">
@@ -196,5 +225,5 @@
         <origin xyz="${base_length / 2.8} 0 -${wheel_radius / 4.0}" rpy="0 0 0" />
     </joint>
-     <!-- Front direction Joint rod-->
+     <!-- Front direction Joint rod
     <joint name="front_direction_link_rod_joint" type="fixed">
         <parent link="base_link" />
@@ -202,4 +231,22 @@
         <origin xyz="${base_length / 2.8} 0 ${base_height}" rpy="0 0 0" />
     </joint>
+     Back direction Joint rod
+    <joint name="back_direction_link_rod_joint" type="fixed">
+        <parent link="base_link" />
+        <child link="back_direction_link_rod" />
+        <origin xyz="-${base_length / 2.8} 0 ${base_height}" rpy="0 0 0" />
+    </joint>
+    left direction Joint rod
+    <joint name="left_direction_link_rod_joint" type="fixed">
+        <parent link="base_link" />
+        <child link="left_direction_link_rod" />
+        <origin xyz="0 -${base_width / 2.5} ${base_height}" rpy="0 0 0" />
+    </joint>
+     right direction Joint rod
+    <joint name="right_direction_link_rod_joint" type="fixed">
+        <parent link="base_link" />
+        <child link="right_direction_link_rod" />
+        <origin xyz="0 ${base_width / 2.5} ${base_height}" rpy="0 0 0" />
+    </joint> -->
     <!-- Back Caster Wheel Joint -->
     <joint name="base_caster_wheel_joint2" type="fixed">

File: install/single_robo_discription/share/single_robo_discription/urdf/mobile_base_gazebo.xacro (robot description, xacro)
@@ -44,5 +44,5 @@
     <sensor name="lidar_sensor" type="gpu_lidar">
       <pose>0 0 0 0 0 0</pose>
-      <update_rate>10</update_rate>
+      <update_rate>30</update_rate>
       <always_on>1</always_on>
       <visualize>true</visualize>
@@ -52,5 +52,5 @@
         <scan>
           <horizontal>
-            <samples>720</samples>
+            <samples>1080</samples>
             <resolution>1</resolution>
             <min_angle>-3.14</min_angle>
@@ -59,6 +59,6 @@
         </scan>
         <range>
-          <min>0.12</min>
-          <max>50.0</max>
+          <min>0.01</min>
+          <max>25.0</max>
           <resolution>0.01</resolution>
         </range>
